File: PCBs/led_driver_1/led_driver_board_1.sch (KiCad schematic (older format))
At the start: 43 parts, among them J10 LED_EN_OUT, J11 PWR_IN, J9 SIG_IN, U5 74HC595, U6 74HC595, U7 74HC595, U8 74HC595

Commit message: Refactor to separate board projects
Parts:
- C12, C13, C14, C15: footprint (none) -> Capacitors_THT:CP_Radial_Tantal_D5.0mm_P2.50mm
- J10: footprint (none) -> Connectors:IDC_Header_Straight_40pins
- J9: footprint (none) -> Connectors:IDC_Header_Straight_8pins
- R14, R15, R16, R17, R18, R19, R20, R21: footprint (none) -> Resistors_THT:R_Axial_DIN0207_L6.3mm_D2.5mm_P10.16mm_Horizontal
- U5, U6, U7, U8: footprint (none) -> Housings_DIP:DIP-14_W7.62mm_Socket
Connections:
- net labels added: LED10_EN_OUT, LED11_EN_OUT, LED12_EN_OUT, LED13_EN_OUT, LED14_EN_OUT, LED15_EN_OUT, LED16_EN_OUT, LED17_EN_OUT, LED18_EN_OUT, LED19_EN_OUT, LED1_EN_OUT, LED20_EN_OUT, LED21_EN_OUT, LED22_EN_OUT, LED23_EN_OUT, LED24_EN_OUT, LED25_EN_OUT, LED26_EN_OUT, LED27_EN_OUT, LED28_EN_OUT, LED29_EN_OUT, LED2_EN_OUT, LED30_EN_OUT, LED31_EN_OUT, LED32_EN_OUT, LED3_EN_OUT, LED4_EN_OUT, LED5_EN_OUT, LED6_EN_OUT, LED7_EN_OUT, LED8_EN_OUT, LED9_EN_OUT
- wire segments 218 -> 250

Commit message: Driver mod and PCB layout
Parts:
- J1: renamed from J11; footprint (none) -> Connectors:PINHEAD1-2
- R10: renamed from R34; footprint (none) -> Resistors_THT:R_Axial_DIN0207_L6.3mm_D2.5mm_P10.16mm_Horizontal
- R12: renamed from R35; footprint (none) -> Resistors_THT:R_Axial_DIN0207_L6.3mm_D2.5mm_P10.16mm_Horizontal
- R14: renamed from R36; footprint (none) -> Resistors_THT:R_Axial_DIN0207_L6.3mm_D2.5mm_P10.16mm_Horizontal
- R16: renamed from R37; footprint (none) -> Resistors_THT:R_Axial_DIN0207_L6.3mm_D2.5mm_P10.16mm_Horizontal
- R17: renamed from R22; footprint (none) -> Resistors_THT:R_Axial_DIN0207_L6.3mm_D2.5mm_P10.16mm_Horizontal
- R18: renamed from R38; footprint (none) -> Resistors_THT:R_Axial_DIN0207_L6.3mm_D2.5mm_P10.16mm_Horizontal
- R19: renamed from R23; footprint (none) -> Resistors_THT:R_Axial_DIN0207_L6.3mm_D2.5mm_P10.16mm_Horizontal
- R2: renamed from R30; footprint (none) -> Resistors_THT:R_Axial_DIN0207_L6.3mm_D2.5mm_P10.16mm_Horizontal
- R20: renamed from R39; footprint (none) -> Resistors_THT:R_Axial_DIN0207_L6.3mm_D2.5mm_P10.16mm_Horizontal
- R21: renamed from R24; footprint (none) -> Resistors_THT:R_Axial_DIN0207_L6.3mm_D2.5mm_P10.16mm_Horizontal
- R22: renamed from R40; footprint (none) -> Resistors_THT:R_Axial_DIN0207_L6.3mm_D2.5mm_P10.16mm_Horizontal
- R23: renamed from R25; footprint (none) -> Resistors_THT:R_Axial_DIN0207_L6.3mm_D2.5mm_P10.16mm_Horizontal
- R24: renamed from R41; footprint (none) -> Resistors_THT:R_Axial_DIN0207_L6.3mm_D2.5mm_P10.16mm_Horizontal
- R25: renamed from R26; footprint (none) -> Resistors_THT:R_Axial_DIN0207_L6.3mm_D2.5mm_P10.16mm_Horizontal
- R26: renamed from R42; footprint (none) -> Resistors_THT:R_Axial_DIN0207_L6.3mm_D2.5mm_P10.16mm_Horizontal
- R27: footprint (none) -> Resistors_THT:R_Axial_DIN0207_L6.3mm_D2.5mm_P10.16mm_Horizontal
- R28: renamed from R43; footprint (none) -> Resistors_THT:R_Axial_DIN0207_L6.3mm_D2.5mm_P10.16mm_Horizontal
- R29: renamed from R28; footprint (none) -> Resistors_THT:R_Axial_DIN0207_L6.3mm_D2.5mm_P10.16mm_Horizontal
- R30: renamed from R44; footprint (none) -> Resistors_THT:R_Axial_DIN0207_L6.3mm_D2.5mm_P10.16mm_Horizontal
- R31: renamed from R29; footprint (none) -> Resistors_THT:R_Axial_DIN0207_L6.3mm_D2.5mm_P10.16mm_Horizontal
- R32: renamed from R45; footprint (none) -> Resistors_THT:R_Axial_DIN0207_L6.3mm_D2.5mm_P10.16mm_Horizontal
- R4: renamed from R31; footprint (none) -> Resistors_THT:R_Axial_DIN0207_L6.3mm_D2.5mm_P10.16mm_Horizontal
- R6: renamed from R32; footprint (none) -> Resistors_THT:R_Axial_DIN0207_L6.3mm_D2.5mm_P10.16mm_Horizontal
- R8: renamed from R33; footprint (none) -> Resistors_THT:R_Axial_DIN0207_L6.3mm_D2.5mm_P10.16mm_Horizontal
- U1: renamed from U5; footprint Housings_DIP:DIP-14_W7.62mm_Socket -> Housings_DIP:DIP-16_W7.62mm_Socket
- U2: renamed from U6; footprint Housings_DIP:DIP-14_W7.62mm_Socket -> Housings_DIP:DIP-16_W7.62mm_Socket
- U3: renamed from U7; footprint Housings_DIP:DIP-14_W7.62mm_Socket -> Housings_DIP:DIP-16_W7.62mm_Socket
- U4: renamed from U8; footprint Housings_DIP:DIP-14_W7.62mm_Socket -> Housings_DIP:DIP-16_W7.62mm_Socket
- renumbered C12 to C1, C14 to C2, C13 to C3, C15 to C4, J9 to J2, J10 to J3, R14 to R1, R19 to R11, R20 to R13, R21 to R15, R15 to R3, R16 to R5, R17 to R7, R18 to R9
Connections:
- net labels added: +5VD
- net labels removed: +5V, LED10_EN_OUT, LED11_EN_OUT, LED12_EN_OUT, LED13_EN_OUT, LED14_EN_OUT, LED15_EN_OUT, LED16_EN_OUT, LED17_EN_OUT, LED18_EN_OUT, LED19_EN_OUT, LED1_EN_OUT, LED20_EN_OUT, LED21_EN_OUT, LED22_EN_OUT, LED23_EN_OUT, LED24_EN_OUT, LED25_EN_OUT, LED26_EN_OUT, LED27_EN_OUT, LED28_EN_OUT, LED29_EN_OUT, LED2_EN_OUT, LED30_EN_OUT, LED31_EN_OUT, LED32_EN_OUT, LED3_EN_OUT, LED4_EN_OUT, LED5_EN_OUT, LED6_EN_OUT, LED7_EN_OUT, LED8_EN_OUT, LED9_EN_OUT, SFT_REG1_SER, SFT_REG2_SER, SFT_REG3_SER, SFT_REG4_SER
- wire segments 250 -> 216
Other:
- moved on the sheet: J1
