File: PCBs/led_driver_2/led_driver_board_2.sch (KiCad schematic (older format))
At the start: 43 parts, among them J12 SIG_IN, J13 PWR_IN, J14 LED_EN_OUT, U10 74HC595, U11 74HC595, U12 74HC595, U9 74HC595

Commit message: Driver mod and PCB layout
Parts:
- renumbered C16 to C1, C17 to C2, C18 to C3, C19 to C4, J12 to J1, J13 to J2, J14 to J3, R46 to R1, R55 to R10, R56 to R11, R57 to R12, R58 to R13, R59 to R14, R60 to R15, R61 to R16, R62 to R17, R63 to R18, R64 to R19, R47 to R2, R65 to R20, R66 to R21, R67 to R22, R68 to R23, R69 to R24, R70 to R25, R71 to R26, R72 to R27, R73 to R28, R74 to R29, R48 to R3, R75 to R30, R76 to R31, R77 to R32, R49 to R4, R50 to R5, R51 to R6, R52 to R7, R53 to R8, R54 to R9, U9 to U1, U10 to U2, U11 to U3, U12 to U4
Connections:
- net LED33_EN_OUT renamed LED33_EN
- net LED34_EN_OUT renamed LED34_EN
- net LED35_EN_OUT renamed LED35_EN
- net LED36_EN_OUT renamed LED36_EN
- net LED37_EN_OUT renamed LED37_EN
- net LED38_EN_OUT renamed LED38_EN
- net LED39_EN_OUT renamed LED39_EN
- net LED40_EN_OUT renamed LED40_EN
- net LED41_EN_OUT renamed LED41_EN
- net LED42_EN_OUT renamed LED42_EN
- net LED43_EN_OUT renamed LED43_EN
- net LED44_EN_OUT renamed LED44_EN
- net LED45_EN_OUT renamed LED45_EN
- net LED46_EN_OUT renamed LED46_EN
- net LED47_EN_OUT renamed LED47_EN
- net LED48_EN_OUT renamed LED48_EN
- net LED49_EN_OUT renamed LED49_EN
- net LED50_EN_OUT renamed LED50_EN
- net LED51_EN_OUT renamed LED51_EN
- net LED52_EN_OUT renamed LED52_EN
- net LED53_EN_OUT renamed LED53_EN
- net LED54_EN_OUT renamed LED54_EN
- net LED55_EN_OUT renamed LED55_EN
- net LED56_EN_OUT renamed LED56_EN
- net LED57_EN_OUT renamed LED57_EN
- net LED58_EN_OUT renamed LED58_EN
- net LED59_EN_OUT renamed LED59_EN
- net LED60_EN_OUT renamed LED60_EN
- net LED61_EN_OUT renamed LED61_EN
- net LED62_EN_OUT renamed LED62_EN
- net LED63_EN_OUT renamed LED63_EN
- net LED64_EN_OUT renamed LED64_EN
- net SFT_REG5_SER renamed SR5_SER
- net SFT_REG6_SER renamed SR6_SER
- net SFT_REG7_SER renamed SR7_SER
